File: base/base_without_battery/base.kicad_pcb (KiCad board)
At the start: 2 copper layers, 84.3 x 50.8 mm, 32 parts, among them J1 USB_B_Micro, J2 Conn_01x06, SW1 SW_Push_Open, SW2 SW_Push_Open, U1 ESP32-WROOM-32, U2 MCP73831-3-OT, U3 BMP280, U4 TPS63001

Commit message: add base finish
Parts:
- removed BT1: 1043, 18650:BAT_1043
- removed C6, C7, C8: 0.1uF, Capacitor_SMD:C_0603_1608Metric
- removed D3: LED, LED_SMD:LED_0603_1608Metric
- removed D4, D5: 1N4007, Diode_SMD:Nexperia_CFP3_SOD-123W
- removed L1: LPS4012-103MRB, LPS4012:IND_LPS4012-103MRB
- removed R7, R8, R9: 100, Resistor_SMD:R_0603_1608Metric
- removed U4: TPS63001, Package_SON:Texas_DRC0010J_ThermalVias
- added C3: C, Capacitor_SMD:C_0603_1608Metric, F.Cu at (97.8, 83.7)
- C1, C2: value 0.1uF -> C
- U2: value MCP73831-3-OT -> LM317_SOT-223; footprint Package_TO_SOT_SMD:SOT-23-5 -> Package_TO_SOT_SMD:SOT-223-3_TabPin2
- moved C2 15.0 mm to (109.1, 89.3), turned to -90 degrees
- moved C1 8.82 mm to (106.9, 89.3), turned to -90 degrees
- moved U2 1.57 mm to (100.8, 88.4)
Connections:
- C1 pad 1: 5V -> VCC
- C2 pad 1: BAT+ -> VCC
- U2 pad 1: Net-(U2-STAT) -> GND
- U2 pad 2: GND -> VCC
- U2 pad 3: BAT+ -> 5V
Routing:
- net BAT+: track 91.7 -> 0.00 mm
- net GND: track 18.7 -> 7.79 mm, vias 31 -> 22
- net Net-(D4-K): track 9.27 -> 0.00 mm
- net Net-(U4-EN): track 6.41 -> 0.00 mm
- net VCC: track 163.4 -> 157.9 mm
- net Net-(U4-L2): track 4.29 -> 0.00 mm
- net Net-(U4-L1): track 4.16 -> 0.00 mm
- net Net-(D3-K): track 2.57 -> 0.00 mm
- net Net-(U2-PROG): track 2.11 -> 0.00 mm
- net Net-(U2-STAT): track 2.09 -> 0.00 mm
- net DW_IRQ: track 74.6 -> 73.2 mm
- net 5V: track 79.9 -> 80.7 mm, vias 3 -> 2
Other:
- board size 84.3 x 50.8 mm -> 84.3 x 34 mm
