File: base/base_without_battery/base.kicad_sch (KiCad schematic)
At the start: 32 parts, among them J1 USB_B_Micro, J2 Conn_01x06, SW1 SW_Push_Open, SW2 SW_Push_Open, U1 ESP32-WROOM-32, U2 MCP73831-3-OT, U3 BMP280, U4 TPS63001

Commit message: add base finish
Parts:
- removed BT1: 1043, 18650:BAT_1043, symbol 18650:1043
- removed C6, C7, C8: 0.1uF, Capacitor_SMD:C_0603_1608Metric, symbol Device:C
- removed D3: LED, LED_SMD:LED_0603_1608Metric, symbol Device:LED
- removed D4, D5: 1N4007, Diode_SMD:Nexperia_CFP3_SOD-123W, symbol Diode:1N4007
- removed L1: LPS4012-103MRB, LPS4012:IND_LPS4012-103MRB, symbol LPS4012:LPS4012-103MRB
- removed R7, R8, R9: 100, Resistor_SMD:R_0603_1608Metric, symbol Device:R_Small
- removed U2: MCP73831-3-OT, Package_TO_SOT_SMD:SOT-23-5, symbol Battery_Management:MCP73831-3-OT
- removed U4: TPS63001, Package_SON:Texas_DRC0010J_ThermalVias, symbol Regulator_Switching:TPS63000
- added C3: C, Capacitor_SMD:C_0603_1608Metric, symbol Device:C
- added U2: LM317_SOT-223, Package_TO_SOT_SMD:SOT-223-3_TabPin2, symbol Regulator_Linear:LM317_SOT-223
- C1, C2: value 0.1uF -> C
Connections:
- net BAT+ is gone; now on net VCC: C2.1
- net 5V: now also C3.1, U2.3 (VI); no longer C1.1
- net GND: now also C3.2, U2.1 (ADJ)
- net VCC: now also C1.1, U2.2 (VO)
